File: pcb/nosepoke.kicad_pcb (KiCad board)
At the start: 2 copper layers, 31 x 21.6 mm, 9 parts, among them J1 0855135013, Q1 PT26-21C/TR8

Commit message: rear pcb v1.16
Parts:
- added R5: 20KΩ, Resistor_SMD:R_0603_1608Metric, F.Cu at (152.9, 102.4)
- R1: value 330Ω -> 200Ω
- moved R3 1.02 mm to (146.8, 97.5), turned to -90 degrees
- moved R2 1.02 mm to (149.9, 99.1)
Connections:
- net /5VDC renamed +5V
- D1 pad 1: GND -> Net-(D1-Pad1)
- J1 pad 7: (no net) -> Net-(D1-Pad1)
Routing:
- net Net-(D1-Pad1): track 0.00 -> 25.0 mm
- net /DIO_A: track 14.4 -> 19.2 mm
- net +5V: track 40.7 -> 37.6 mm
- net Net-(D2-Pad2): track 3.52 -> 4.41 mm
Other:
- net class Default removed
- rule pad_to_mask_clearance: 0.051 -> 0
- board text added: "Nosepoke v1.16"
- board text removed: "Nosepoke v1.15"

Commit message: backside PCB v1.17
Parts:
- H1, H2: footprint asl_footprints:MountingHole_2.7mm_M2.5 -> MountingHole:MountingHole_2.7mm_M2.5_DIN965_Pad_TopOnly
- renumbered R3 to R2, R2 to R3, R5 to R4
Connections:
- J1 pad 4: (no net) -> unconnected-(J1-Pad4)
- J1 pad 5: (no net) -> unconnected-(J1-Pad5)
- J1 pad 8: (no net) -> unconnected-(J1-Pad8)
Other:
- board text added: "Nosepoke v1.17"
- board text removed: "Nosepoke v1.16"
