File: pcb/side_emitter_detector.kicad_pcb (KiCad board)
At the start: 2 copper layers, 23 x 6.4 mm, 5 parts, among them J1 Conn_01x02_Male

Commit message: backside PCB v1.17
Other:
- net class Default removed
